Commit message: Backup de cambios en FUERTE

File: Sources/summit/summit_sim/summit_description/urdf/summit.urdf (robot description, URDF)
Before this commit: robot summit, 13 links, 12 joints
Links:
- removed link hokuyo_laser_box_link
- removed link hokuyo_laser_link
- added link rplidar_laser_box_link, mass 0.01; collision box size=0.05 0.05 0.1; visual box size=0.05 0.05 0.1
- added link rplidar_laser_link, mass 0.001
Joints:
- removed joint hokuyo_laser_box_joint
- removed joint hokuyo_laser_joint
- added joint rplidar_laser_box_joint: type fixed, parent rplidar_laser_link, child rplidar_laser_box_link, origin xyz=0 0 0 rpy=0 0 0
- added joint rplidar_laser_joint: type fixed, parent base_link, child rplidar_laser_link, origin xyz=0.01 0 0.24 rpy=0 0 -3.15, axis 0 1 0
