Commit message: subo todos los cambios de quique a dia de hoy

File: Sources/summit_sim/summit_description/urdf/summit.urdf.xacro (robot description, xacro)
@@ -98,8 +98,8 @@
     <parent link="base_link"/>
     <child link="back_left_wheel_dir"/>
-    <origin xyz="-${wheel_offset_x} ${wheel_offset_y} 0" rpy="0 0 0" />
+    <origin xyz="-0.185 0.105 0" rpy="0 0 0" />
     <axis xyz="0 0 1" rpy="0 0 0" />
-    <limit effort="${steer_joint_effort_limit}" velocity="${steer_joint_velocity_limit}" lower="-0.7854" upper="0.7854"/>
-    <joint_properties damping="${steer_joint_damping}" friction="{steer_joint_friction}"/>
+    <limit effort="100.0" velocity="3.0" lower="-0.7854" upper="0.7854"/>
+    <joint_properties damping="0.2" friction="0.1"/>
   </joint>
   <transmission name="joint_blw_trans_dir">
@@ -108,5 +108,5 @@
     <actuator name="joint_blw_motor_dir">
 	  <hardwareInterface>EffortJointInterface</hardwareInterface>
-      <mechanicalReduction>${steer_mechanical_reduction}</mechanicalReduction>
+      <mechanicalReduction>100.0</mechanicalReduction>
 	  <!-- motorTorqueConstant>1</motorTorqueConstant -->
 	</actuator>
@@ -140,6 +140,6 @@
     <origin xyz="0.0 0.060 0" rpy="0 0 0" />
     <axis xyz="0 1 0" rpy="0 0 0" />
-    <limit effort="${wheel_joint_effort_limit}" velocity="${wheel_joint_velocity_limit}"/>
-    <joint_properties damping="${wheel_joint_damping}" friction="{wheel_joint_friction}"/>
+    <limit effort="100.0" velocity="200.0"/>
+    <joint_properties damping="0.0" friction="0.0"/>
   </joint>
   <transmission name="joint_blw_trans">
@@ -148,5 +148,5 @@
      <actuator name="joint_blw_motor">
 	    <hardwareInterface>VelocityJointInterface</hardwareInterface>
-        <mechanicalReduction>${wheel_mechanical_reduction}</mechanicalReduction>
+        <mechanicalReduction>100.0</mechanicalReduction>
      	<!-- motorTorqueConstant>1</motorTorqueConstant -->
 	 </actuator>
@@ -179,8 +179,8 @@
     <parent link="base_link"/>
     <child link="back_right_wheel_dir"/>
-    <origin xyz="-${wheel_offset_x} -${wheel_offset_y} 0" rpy="0 0 0" />
+    <origin xyz="-0.185 -0.105 0" rpy="0 0 0" />
     <axis xyz="0 0 1" rpy="0 0 0" />
-    <limit effort="${steer_joint_effort_limit}" velocity="${steer_joint_velocity_limit}" lower="-0.7854" upper="0.7854"/>
-    <joint_properties damping="${steer_joint_damping}" friction="{steer_joint_friction}"/>
+    <limit effort="100.0" velocity="3.0" lower="-0.7854" upper="0.7854"/>
+    <joint_properties damping="0.2" friction="0.1"/>
   </joint>
   <transmission name="joint_brw_trans_dir">
@@ -189,5 +189,5 @@
     <actuator name="joint_brw_motor_dir">
 	  <hardwareInterface>EffortJointInterface</hardwareInterface>
-      <mechanicalReduction>${steer_mechanical_reduction}</mechanicalReduction>
+      <mechanicalReduction>100.0</mechanicalReduction>
 	  <!-- motorTorqueConstant>1</motorTorqueConstant -->
 	</actuator>
@@ -221,6 +221,6 @@
     <origin xyz="0.0 -0.060 0" rpy="0 0 0" />
     <axis xyz="0 1 0" rpy="0 0 0" />
-    <limit effort="${wheel_joint_effort_limit}" velocity="${wheel_joint_velocity_limit}"/>
-    <joint_properties damping="${wheel_joint_damping}" friction="{wheel_joint_friction}"/>
+    <limit effort="100.0" velocity="200.0"/>
+    <joint_properties damping="0.0" friction="0.0"/>
   </joint>
   <transmission name="joint_brw_trans">
@@ -229,5 +229,5 @@
      <actuator name="joint_brw_motor">
 	    <hardwareInterface>VelocityJointInterface</hardwareInterface>
-        <mechanicalReduction>${wheel_mechanical_reduction}</mechanicalReduction>
+        <mechanicalReduction>1.0</mechanicalReduction>
      	<!-- motorTorqueConstant>1</motorTorqueConstant -->
 	 </actuator>
@@ -260,8 +260,8 @@
     <parent link="base_link"/>
     <child link="front_left_wheel_dir"/>
-    <origin xyz="${wheel_offset_x} ${wheel_offset_y} 0" rpy="0 0 0" />
+    <origin xyz="0.185 0.105 0" rpy="0 0 0" />
     <axis xyz="0 0 1" rpy="0 0 0" />
-    <limit effort="${steer_joint_effort_limit}" velocity="${steer_joint_velocity_limit}" lower="-0.7854" upper="0.7854"/>
-    <joint_properties damping="${steer_joint_damping}" friction="{steer_joint_friction}"/>
+    <limit effort="100.0" velocity="3.0" lower="-0.7854" upper="0.7854"/>
+    <joint_properties damping="0.2" friction="0.1"/>
   </joint>
   <transmission name="joint_flw_trans_dir">
@@ -270,5 +270,5 @@
     <actuator name="joint_flw_motor_dir">
 	  <hardwareInterface>EffortJointInterface</hardwareInterface>
-      <mechanicalReduction>${steer_mechanical_reduction}</mechanicalReduction>
+      <mechanicalReduction>100.0</mechanicalReduction>
 	  <!-- motorTorqueConstant>1</motorTorqueConstant -->
 	</actuator>
@@ -302,6 +302,6 @@
     <origin xyz="0.0 0.060 0" rpy="0 0 0" />
     <axis xyz="0 1 0" rpy="0 0 0" />
-    <limit effort="${wheel_joint_effort_limit}" velocity="${wheel_joint_velocity_limit}"/>
-    <joint_properties damping="${wheel_joint_damping}" friction="{wheel_joint_friction}"/>
+    <limit effort="100.0" velocity="200.0"/>
+    <joint_properties damping="0.0" friction="0.0"/>
   </joint>
   <transmission name="joint_flw_trans">
@@ -310,5 +310,5 @@
      <actuator name="joint_flw_motor">
 	    <hardwareInterface>VelocityJointInterface</hardwareInterface>
-        <mechanicalReduction>${wheel_mechanical_reduction}</mechanicalReduction>
+        <mechanicalReduction>1.0</mechanicalReduction>
      	<!-- motorTorqueConstant>1</motorTorqueConstant -->
 	 </actuator>
@@ -341,8 +341,8 @@
     <parent link="base_link"/>
     <child link="front_right_wheel_dir"/>
-    <origin xyz="${wheel_offset_x} -${wheel_offset_y} 0" rpy="0 0 0" />
+    <origin xyz="0.185 -0.105 0" rpy="0 0 0" />
     <axis xyz="0 0 1" rpy="0 0 0" />
-    <limit effort="${steer_joint_effort_limit}" velocity="${steer_joint_velocity_limit}" lower="-0.7854" upper="0.7854"/>
-    <joint_properties damping="${steer_joint_damping}" friction="{steer_joint_friction}"/>
+    <limit effort="100.0" velocity="3.0" lower="-0.7854" upper="0.7854"/>
+    <joint_properties damping="0.2" friction="0.1"/>
   </joint>
   <transmission name="joint_frw_trans_dir">
@@ -351,5 +351,5 @@
     <actuator name="joint_frw_motor_dir">
 	  <hardwareInterface>EffortJointInterface</hardwareInterface>
-      <mechanicalReduction>${steer_mechanical_reduction}</mechanicalReduction>
+      <mechanicalReduction>100.0</mechanicalReduction>
 	  <!-- motorTorqueConstant>1</motorTorqueConstant -->
 	</actuator>
@@ -383,6 +383,6 @@
     <origin xyz="0.0 -0.060 0" rpy="0 0 0" />
     <axis xyz="0 1 0" rpy="0 0 0" />
-    <limit effort="${wheel_joint_effort_limit}" velocity="${wheel_joint_velocity_limit}"/>
-    <joint_properties damping="${wheel_joint_damping}" friction="{wheel_joint_friction}"/>
+    <limit effort="100.0" velocity="200.0"/>
+    <joint_properties damping="0.0" friction="0.0"/>
   </joint>
   <transmission name="joint_frw_trans">
@@ -391,16 +391,16 @@
      <actuator name="joint_frw_motor">
 	    <hardwareInterface>VelocityJointInterface</hardwareInterface>
-        <mechanicalReduction>${wheel_mechanical_reduction}</mechanicalReduction>
+        <mechanicalReduction>1.0</mechanicalReduction>
      	<!-- motorTorqueConstant>1</motorTorqueConstant -->
 	 </actuator>
   </transmission>
-  <!-- HOKUYO SENSOR -->
-  <joint name="hokuyo_laser_joint" type="fixed">
+  <!-- RPLIDAR LASER -->
+  <joint name="rplidar_laser_joint" type="fixed">
      <axis xyz="0 1 0" />
-     <origin xyz="0.226 0 0.120"/>
+     <origin xyz="0.01 0 0.24" rpy="0 0 -3.15"/>
      <parent link="base_link"/>
-     <child link="hokuyo_laser_link"/>
-  </joint>
-  <link name="hokuyo_laser_link" type="laser">
+     <child link="rplidar_laser_link"/>
+  </joint>
+  <link name="rplidar_laser_link" type="laser">
     <collision>
       <origin xyz="0 0 0" rpy="0 0 0"/>
@@ -454,4 +454,10 @@
        <inertia ixx="0.1" ixy="0" ixz="0" iyy="0.1" iyz="0" izz="0.1" />
     </inertial>
+    <visual>
+      <origin rpy="0 0 0" xyz="0 0 0"/>
+      <geometry>
+        <box size="0.001 0.001 0.001"/>
+      </geometry>
+    </visual>
   </link>
   <joint name="joint_camera" type="fixed">
@@ -465,4 +471,5 @@
      <inertial>
        <mass value="0.1" />
+       <!-- origin xyz="0 0 0" rpy="0 0 0" / -->
        <origin xyz="0 0 0" rpy="0 0 0" />
        <inertia ixx="0.1" ixy="0" ixz="0" iyy="0.1" iyz="0" izz="0.1" />
@@ -474,6 +481,6 @@
      <parent link="camera_base_link"/>
      <child link="camera_pan_link"/>
-     <limit effort="${ptz_joint_effort_limit}" velocity="${ptz_joint_velocity_limit}" lower="-3.1416" upper="3.1416"/>
-     <joint_properties damping="${ptz_joint_damping}" friction="{ptz_joint_friction}"/>
+     <limit effort="100.0" velocity="100.0" lower="-3.1416" upper="3.1416"/>
+     <joint_properties damping="0.1" friction="0.1"/>
   </joint>
   <transmission name="joint_pan_trans">
@@ -482,5 +489,5 @@
      <actuator name="pan_motor">
 	   <hardwareInterface>EffortJointInterface</hardwareInterface>
-       <mechanicalReduction>${ptz_mechanical_reduction}</mechanicalReduction>
+       <mechanicalReduction>1.0</mechanicalReduction>
      </actuator>
   </transmission>
@@ -498,6 +505,6 @@
      <parent link="camera_pan_link"/>
      <child link="camera_tilt_link"/>
-     <limit effort="${ptz_joint_effort_limit}" velocity="${ptz_joint_velocity_limit}" lower="-1.5708" upper="1.5708"/>
-     <joint_properties damping="${ptz_joint_damping}" friction="{ptz_joint_friction}"/>
+     <limit effort="100.0" velocity="100.0" lower="-1.5708" upper="1.5708"/>
+     <joint_properties damping="0.1" friction="0.1"/>
   </joint>
   <transmission name="joint_tilt_trans">
@@ -506,5 +513,5 @@
      <actuator name="tilt_motor">
 	   <hardwareInterface>EffortJointInterface</hardwareInterface>
-       <mechanicalReduction>${ptz_mechanical_reduction}</mechanicalReduction>
+       <mechanicalReduction>1.0</mechanicalReduction>
      </actuator>
   </transmission>
