Commit message: Creado dir de papers; modificaciones varias.

File: summit_sim/summit_description/urdf/summit.urdf.xacro (robot description, xacro)
@@ -398,6 +398,6 @@
   <joint name="rplidar_laser_joint" type="fixed">
      <axis xyz="0 1 0" />
-     <origin xyz="0.01 0 0.24" rpy="0 0 -3.15"/>
-     <parent link="base_link"/>
+     <origin xyz="-0.15 0 0.24" rpy="0 0 0"/>
+     <parent link="base_footprint"/>
      <child link="rplidar_laser_link"/>
   </joint>
@@ -420,30 +420,4 @@
       <inertia ixx="1e-6" ixy="0" ixz="0" iyy="1e-6" iyz="0" izz="1e-6" />
     </inertial>
-  </link>
-  <!-- IMU SENSOR -->
-  <joint name="imu_joint" type="fixed">
-      <axis xyz="1 0 0"/> <!-- 0 1 0 -->
-      <origin xyz="0 0 0.2825"/>
-      <parent link="base_link"/>
-      <child link="imu_link"/>
-  </joint>
-  <link name="imu_link">
-      <inertial>
-        <mass value="0.001"/>
-        <origin rpy="0 0 0" xyz="0 0 0"/>
-        <inertia ixx="0.0001" ixy="0" ixz="0" iyy="0.000001" iyz="0" izz="0.0001"/>
-      </inertial>
-      <visual>
-        <origin rpy="0 0 0" xyz="0 0 0"/>
-        <geometry>
-          <box size="0.001 0.001 0.001"/>
-        </geometry>
-      </visual>
-      <collision>
-        <origin rpy="0 0 0" xyz="0 0 0"/>
-        <geometry>
-          <box size=".001 .001 .001"/>
-        </geometry>
-      </collision>
   </link>
   <!-- AXIS PTZ CAMERA WITH PAN AND TILT -->

Commit message: Update the transmission for every joint (EffortJointInterface & VelocityJointInterface)

File: summit_sim/summit_description/urdf/summit.urdf.xacro (robot description, xacro)
@@ -104,4 +104,16 @@
   </joint>
   <transmission name="joint_blw_trans_dir">
+    <type>transmission_interface/SimpleTransmission</type>
+    <joint name="joint_back_left_wheel_dir">
+      <hardwareInterface>hardware_interface/EffortJointInterface</hardwareInterface>
+    </joint>
+    <actuator name="joint_blw_motor_dir">
+      <hardwareInterface>hardware_interface/EffortJointInterface</hardwareInterface>
+      <mechanicalReduction>100.0</mechanicalReduction>
+      <!--motorTorqueConstant>1</motorTorqueConstant-->
+    </actuator>
+  </transmission>
+<!--
+  <transmission name="joint_blw_trans_dir">
 	<type>transmission_interface/SimpleTransmission</type>
     <joint name="joint_back_left_wheel_dir" />
@@ -109,7 +121,8 @@
 	  <hardwareInterface>EffortJointInterface</hardwareInterface>
       <mechanicalReduction>100.0</mechanicalReduction>
-	  <!-- motorTorqueConstant>1</motorTorqueConstant -->
+	   motorTorqueConstant>1</motorTorqueConstant
 	</actuator>
   </transmission>
+-->
   <!-- BACK LEFT WHEEL -->
   <link name="back_left_wheel">
@@ -144,4 +157,16 @@
   </joint>
   <transmission name="joint_blw_trans">
+    <type>transmission_interface/SimpleTransmission</type>
+    <joint name="joint_back_left_wheel">
+      <hardwareInterface>hardware_interface/VelocityJointInterface</hardwareInterface>
+    </joint>
+    <actuator name="joint_blw_motor">
+      <hardwareInterface>hardware_interface/VelocityJointInterface</hardwareInterface>
+      <mechanicalReduction>100.0</mechanicalReduction>
+      <!--motorTorqueConstant>1</motorTorqueConstant-->
+    </actuator>
+  </transmission>
+<!--
+  <transmission name="joint_blw_trans">
 	 <type>transmission_interface/SimpleTransmission</type>
      <joint name="joint_back_left_wheel" />
@@ -149,7 +174,8 @@
 	    <hardwareInterface>VelocityJointInterface</hardwareInterface>
         <mechanicalReduction>100.0</mechanicalReduction>
-     	<!-- motorTorqueConstant>1</motorTorqueConstant -->
+     	< motorTorqueConstant>1</motorTorqueConstant >
 	 </actuator>
   </transmission>
+-->
 <!-- DIRECTION BACK RIGHT        -->
 <!-- =========================== -->
@@ -185,11 +211,13 @@
   </joint>
   <transmission name="joint_brw_trans_dir">
-	<type>transmission_interface/SimpleTransmission</type>
-    <joint name="joint_back_right_wheel_dir" />
+    <type>transmission_interface/SimpleTransmission</type>
+    <joint name="joint_back_right_wheel_dir">
+      <hardwareInterface>hardware_interface/EffortJointInterface</hardwareInterface>
+    </joint>
     <actuator name="joint_brw_motor_dir">
-	  <hardwareInterface>EffortJointInterface</hardwareInterface>
-      <mechanicalReduction>100.0</mechanicalReduction>
-	  <!-- motorTorqueConstant>1</motorTorqueConstant -->
-	</actuator>
+      <hardwareInterface>hardware_interface/EffortJointInterface</hardwareInterface>
+      <mechanicalReduction>100.0</mechanicalReduction>
+      <!--motorTorqueConstant>1</motorTorqueConstant-->
+    </actuator>
   </transmission>
   <!-- BACK RIGHT WHEEL -->
@@ -225,11 +253,13 @@
   </joint>
   <transmission name="joint_brw_trans">
-	 <type>transmission_interface/SimpleTransmission</type>
-     <joint name="joint_back_right_wheel" />
-     <actuator name="joint_brw_motor">
-	    <hardwareInterface>VelocityJointInterface</hardwareInterface>
-        <mechanicalReduction>1.0</mechanicalReduction>
-     	<!-- motorTorqueConstant>1</motorTorqueConstant -->
-	 </actuator>
+    <type>transmission_interface/SimpleTransmission</type>
+    <joint name="joint_back_right_wheel">
+      <hardwareInterface>hardware_interface/VelocityJointInterface</hardwareInterface>
+    </joint>
+    <actuator name="joint_brw_motor">
+      <hardwareInterface>hardware_interface/VelocityJointInterface</hardwareInterface>
+      <mechanicalReduction>100.0</mechanicalReduction>
+      <!--motorTorqueConstant>1</motorTorqueConstant-->
+    </actuator>
   </transmission>
 <!-- DIRECTION FORWARD LEFT      -->
@@ -266,11 +296,13 @@
   </joint>
   <transmission name="joint_flw_trans_dir">
-	<type>transmission_interface/SimpleTransmission</type>
-    <joint name="joint_front_left_wheel_dir" />
+    <type>transmission_interface/SimpleTransmission</type>
+    <joint name="joint_front_left_wheel_dir">
+      <hardwareInterface>hardware_interface/EffortJointInterface</hardwareInterface>
+    </joint>
     <actuator name="joint_flw_motor_dir">
-	  <hardwareInterface>EffortJointInterface</hardwareInterface>
-      <mechanicalReduction>100.0</mechanicalReduction>
-	  <!-- motorTorqueConstant>1</motorTorqueConstant -->
-	</actuator>
+      <hardwareInterface>hardware_interface/EffortJointInterface</hardwareInterface>
+      <mechanicalReduction>100.0</mechanicalReduction>
+      <!--motorTorqueConstant>1</motorTorqueConstant-->
+    </actuator>
   </transmission>
   <!-- FRONT LEFT WHEEL (GREY) -->
@@ -306,11 +338,13 @@
   </joint>
   <transmission name="joint_flw_trans">
-	 <type>transmission_interface/SimpleTransmission</type>
-     <joint name="joint_front_left_wheel" />
-     <actuator name="joint_flw_motor">
-	    <hardwareInterface>VelocityJointInterface</hardwareInterface>
-        <mechanicalReduction>1.0</mechanicalReduction>
-     	<!-- motorTorqueConstant>1</motorTorqueConstant -->
-	 </actuator>
+    <type>transmission_interface/SimpleTransmission</type>
+    <joint name="joint_front_left_wheel">
+      <hardwareInterface>hardware_interface/VelocityJointInterface</hardwareInterface>
+    </joint>
+    <actuator name="joint_flw_motor">
+      <hardwareInterface>hardware_interface/VelocityJointInterface</hardwareInterface>
+      <mechanicalReduction>100.0</mechanicalReduction>
+      <!--motorTorqueConstant>1</motorTorqueConstant-->
+    </actuator>
   </transmission>
 <!-- DIRECTION FORWARD RIGHT     -->
@@ -347,11 +381,13 @@
   </joint>
   <transmission name="joint_frw_trans_dir">
-	<type>transmission_interface/SimpleTransmission</type>
-    <joint name="joint_front_right_wheel_dir" />
+    <type>transmission_interface/SimpleTransmission</type>
+    <joint name="joint_front_right_wheel_dir">
+      <hardwareInterface>hardware_interface/EffortJointInterface</hardwareInterface>
+    </joint>
     <actuator name="joint_frw_motor_dir">
-	  <hardwareInterface>EffortJointInterface</hardwareInterface>
-      <mechanicalReduction>100.0</mechanicalReduction>
-	  <!-- motorTorqueConstant>1</motorTorqueConstant -->
-	</actuator>
+      <hardwareInterface>hardware_interface/EffortJointInterface</hardwareInterface>
+      <mechanicalReduction>100.0</mechanicalReduction>
+      <!--motorTorqueConstant>1</motorTorqueConstant-->
+    </actuator>
   </transmission>
   <!-- FRONT RIGHT WHEEL (GREY) -->
@@ -387,11 +423,13 @@
   </joint>
   <transmission name="joint_frw_trans">
-	 <type>transmission_interface/SimpleTransmission</type>
-     <joint name="joint_front_right_wheel" />
-     <actuator name="joint_frw_motor">
-	    <hardwareInterface>VelocityJointInterface</hardwareInterface>
-        <mechanicalReduction>1.0</mechanicalReduction>
-     	<!-- motorTorqueConstant>1</motorTorqueConstant -->
-	 </actuator>
+    <type>transmission_interface/SimpleTransmission</type>
+    <joint name="joint_front_right_wheel">
+      <hardwareInterface>hardware_interface/VelocityJointInterface</hardwareInterface>
+    </joint>
+    <actuator name="joint_frw_motor">
+      <hardwareInterface>hardware_interface/VelocityJointInterface</hardwareInterface>
+      <mechanicalReduction>100.0</mechanicalReduction>
+      <!--motorTorqueConstant>1</motorTorqueConstant-->
+    </actuator>
   </transmission>
   <!-- LASER SENSOR -->
@@ -400,7 +438,7 @@
      <origin xyz="0 0 0.24" rpy="0 0 0"/>
      <parent link="base_footprint"/>
-     <child link="laser_link"/>
-  </joint>
-  <link name="laser_link" type="laser">
+     <child link="hokuyo_laser_link"/>
+  </joint>
+  <link name="hokuyo_laser_link" type="laser">
     <collision>
       <origin xyz="0 0 0" rpy="0 0 0"/>
@@ -459,10 +497,12 @@
   </joint>
   <transmission name="joint_pan_trans">
-	 <type>transmission_interface/SimpleTransmission</type>
-     <joint name="joint_camera_pan" />
-     <actuator name="pan_motor">
-	   <hardwareInterface>EffortJointInterface</hardwareInterface>
-       <mechanicalReduction>1.0</mechanicalReduction>
-     </actuator>
+    <type>transmission_interface/SimpleTransmission</type>
+    <joint name="joint_camera_pan">
+      <hardwareInterface>hardware_interface/EffortJointInterface</hardwareInterface>
+    </joint>
+    <actuator name="pan_motor">
+      <hardwareInterface>hardware_interface/EffortJointInterface</hardwareInterface>
+      <mechanicalReduction>1.0</mechanicalReduction>
+    </actuator>
   </transmission>
   <link name="camera_tilt_link">
@@ -483,10 +523,12 @@
   </joint>
   <transmission name="joint_tilt_trans">
-	 <type>transmission_interface/SimpleTransmission</type>
-     <joint name="joint_camera_tilt" />
-     <actuator name="tilt_motor">
-	   <hardwareInterface>EffortJointInterface</hardwareInterface>
-       <mechanicalReduction>1.0</mechanicalReduction>
-     </actuator>
+    <type>transmission_interface/SimpleTransmission</type>
+    <joint name="joint_camera_tilt">
+      <hardwareInterface>hardware_interface/EffortJointInterface</hardwareInterface>
+    </joint>
+    <actuator name="tilt_motor">
+      <hardwareInterface>hardware_interface/EffortJointInterface</hardwareInterface>
+      <mechanicalReduction>1.0</mechanicalReduction>
+    </actuator>
   </transmission>
 </robot>

Commit message: Modified Hokuyo in the simulation with its base and removed camera...

File: summit_sim/summit_description/urdf/summit.urdf.xacro (robot description, xacro)
@@ -63,5 +63,5 @@
     </visual>
     <collision>
-       <origin xyz="0 0 0.06" rpy="0 0 0 " />
+       <origin xyz="0 0 0" rpy="0 0 0 " />
        <geometry>
          <mesh filename="package://summit_description/meshes/summit_chassis.dae"/>
@@ -349,5 +349,5 @@
   </transmission>
 <!-- DIRECTION FORWARD RIGHT     -->
-<!-- =========================== -->
+<!-- =================================================================== -->
   <link name="front_right_wheel_dir">
     <inertial>
@@ -391,4 +391,5 @@
     </actuator>
   </transmission>
+  <!-- =================================================================== -->
   <!-- FRONT RIGHT WHEEL (GREY) -->
   <link name="front_right_wheel">
@@ -433,24 +434,50 @@
     </actuator>
   </transmission>
+  <!-- =================================================================== -->
+  <!-- SOPORTE LASER  -->
+  <joint name="base_laser_joint" type="fixed">
+    <origin xyz="-0.25 0 0.29" rpy="0 0 0"/>
+    <parent link="base_footprint"/>
+    <child link="hokuyo_base_link"/>
+  </joint>
+  <link name="hokuyo_base_link">
+    <visual>
+      <origin xyz="-0.02 -0.03 -0.01" rpy="${PI/2} 0 ${PI/2}"/>
+      <geometry>
+        <mesh filename="package://summit_description/meshes/soporte_laser.STL" scale="0.001 0.001 0.001"/>
+      </geometry>
+    </visual>
+    <collision>
+      <origin xyz="-0.02 -0.03 -0.01" rpy="${PI/2} 0 ${PI/2}"/>
+      <geometry>
+        <mesh filename="package://summit_description/meshes/soporte_laser.STL" scale="0.001 0.001 0.001"/>
+      </geometry>
+    </collision>
+    <inertial>
+      <mass value="1" />
+      <origin xyz="0 0 0" rpy="0 0 0"/>
+      <inertia ixx="1" ixy="0" ixz="0" iyy="1" iyz="0" izz="1" />
+    </inertial>
+  </link>
+  <!-- =================================================================== -->
   <!-- LASER SENSOR -->
   <joint name="laser_joint" type="fixed">
-     <axis xyz="0 1 0" />
-     <origin xyz="0 0 0.24" rpy="0 0 0"/>
-     <parent link="base_footprint"/>
+     <origin xyz="0 0 0.05" rpy="0 0 0"/>
+     <parent link="hokuyo_base_link"/>
      <child link="hokuyo_laser_link"/>
   </joint>
   <link name="hokuyo_laser_link" type="laser">
-    <collision>
-      <origin xyz="0 0 0" rpy="0 0 0"/>
+    <visual>
+      <origin xyz="-0.02 -0.025 0" rpy="${PI/2} 0 ${PI/2}"/>
       <geometry>
-	     <box size="0.1 0.1 0.1"/>
+        <mesh filename="package://summit_description/meshes/Hokuyo_UST-10LX.STL" scale="0.001 0.001 0.001"/>
       </geometry>
-    </collision>
-    <visual>
-      <origin xyz="0 0 0" rpy="0 0 0"/>
+    </visual>
+    <collision>
+      <origin xyz="-0.02 -0.025 0" rpy="${PI/2} 0 ${PI/2}"/>
       <geometry>
-        <mesh filename="package://summit_description/meshes/hokuyo-utm30-lx.dae"/>
+        <mesh filename="package://summit_description/meshes/Hokuyo_UST-10LX.STL" scale="0.001 0.001 0.001"/>
       </geometry>
-    </visual>
+    </collision>
     <inertial>
       <mass value="1e-5" />
@@ -459,5 +486,7 @@
     </inertial>
   </link>
+  <!-- =================================================================== -->
   <!-- AXIS PTZ CAMERA WITH PAN AND TILT -->
+  <!--
   <link name="camera_base_link">
      <inertial>
@@ -475,5 +504,4 @@
   <joint name="joint_camera" type="fixed">
      <axis xyz="0 1 0" />
-     <!--origin xyz="0.180 0.0 0.270"/-->
      <origin xyz="0.150 0.0 0.240"/>
      <parent link="base_link"/>
@@ -483,5 +511,4 @@
      <inertial>
        <mass value="0.1" />
-       <!-- origin xyz="0 0 0" rpy="0 0 0" / -->
        <origin xyz="0 0 0" rpy="0 0 0" />
        <inertia ixx="0.1" ixy="0" ixz="0" iyy="0.1" iyz="0" izz="0.1" />
@@ -509,5 +536,4 @@
      <inertial>
        <mass value="0.1" />
-       <!-- origin xyz="0 0 0" rpy="0 0 0" / -->
        <origin xyz="0 0 0.3" rpy="0 0 0" />
        <inertia ixx="0.1" ixy="0" ixz="0" iyy="0.1" iyz="0" izz="0.1" />
@@ -532,3 +558,4 @@
     </actuator>
   </transmission>
+-->
 </robot>

Commit message: Asus (xtion pro live) partially integrated in the simulation.

File: summit_sim/summit_description/urdf/summit.urdf.xacro (robot description, xacro)
@@ -437,6 +437,6 @@
   <!-- SOPORTE LASER  -->
   <joint name="base_laser_joint" type="fixed">
-    <origin xyz="-0.25 0 0.29" rpy="0 0 0"/>
-    <parent link="base_footprint"/>
+    <origin xyz="-0.25 0 0.24" rpy="0 0 0"/>
+    <parent link="base_link"/>
     <child link="hokuyo_base_link"/>
   </joint>
@@ -463,7 +463,7 @@
   <!-- LASER SENSOR -->
   <joint name="laser_joint" type="fixed">
-     <origin xyz="0 0 0.05" rpy="0 0 0"/>
      <parent link="hokuyo_base_link"/>
      <child link="hokuyo_laser_link"/>
+     <origin xyz="0 0 0.05" rpy="0 0 0"/>
   </joint>
   <link name="hokuyo_laser_link" type="laser">
@@ -487,6 +487,27 @@
   </link>
   <!-- =================================================================== -->
+  <!-- ASUS xtion_pro_live -->
+  <joint name="joint_camera" type="fixed">
+     <parent link="base_link"/>
+     <child link="camera_link"/>
+     <origin xyz="0.08 0.0 0.265" rpy="0 0 0"/>
+  </joint>
+  <link name="camera_link">
+    <visual>
+      <origin xyz="0 0 0" rpy="0 0 0"/>
+      <geometry>
+        <mesh filename="package://summit_description/meshes/xtion_pro_live.dae" />
+      </geometry>
+    </visual>
+    <collision>
+      <origin xyz="0 0 0" rpy="0 0 0"/>
+      <geometry>
+        <mesh filename="package://summit_description/meshes/xtion_pro_live.dae" />
+      </geometry>
+    </collision>
+  </link>
+  <!-- =================================================================== -->
   <!-- AXIS PTZ CAMERA WITH PAN AND TILT -->
-  <!--
+<!--
   <link name="camera_base_link">
      <inertial>
@@ -496,5 +517,5 @@
     </inertial>
     <visual>
-      <origin rpy="0 0 0" xyz="0 0 0"/>
+      <origin rpy="0 0 0" xyz="0 0 0.2"/>
       <geometry>
         <box size="0.001 0.001 0.001"/>

Commit message: Fixed Hokuyo laser TF

File: summit_sim/summit_description/urdf/summit.urdf.xacro (robot description, xacro)
@@ -3,4 +3,6 @@
   <!-- Import all Gazebo-customization elements, including Gazebo colors -->
   <xacro:include filename="$(find summit_description)/urdf/summit.gazebo" />
+  <!-- Import Rviz colors -->
+	<xacro:include filename="$(find summit_description)/urdf/materials.xacro" />
   <!-- Robot mechanical and motor parameters -->
   <xacro:property name="PI" value="3.1415926535897931"/>
@@ -447,4 +449,5 @@
         <mesh filename="package://summit_description/meshes/soporte_laser.STL" scale="0.001 0.001 0.001"/>
       </geometry>
+      <material name="Blue" />
     </visual>
     <collision>
@@ -465,15 +468,16 @@
      <parent link="hokuyo_base_link"/>
      <child link="hokuyo_laser_link"/>
-     <origin xyz="0 0 0.05" rpy="0 0 0"/>
+     <origin xyz="0.01 0 0.099" rpy="0 0 0"/>
   </joint>
   <link name="hokuyo_laser_link" type="laser">
     <visual>
-      <origin xyz="-0.02 -0.025 0" rpy="${PI/2} 0 ${PI/2}"/>
+      <origin xyz="-0.033 -0.025 -0.05" rpy="${PI/2} 0 ${PI/2}"/>
       <geometry>
         <mesh filename="package://summit_description/meshes/Hokuyo_UST-10LX.STL" scale="0.001 0.001 0.001"/>
       </geometry>
-    </visual>
-    <collision>
-      <origin xyz="-0.02 -0.025 0" rpy="${PI/2} 0 ${PI/2}"/>
+      <material name="light_grey" />
+    </visual>
+    <collision>
+      <origin xyz="-0.033 -0.025 -0.04" rpy="${PI/2} 0 ${PI/2}"/>
       <geometry>
         <mesh filename="package://summit_description/meshes/Hokuyo_UST-10LX.STL" scale="0.001 0.001 0.001"/>

Commit message: Modification in camera's TF

File: summit_sim/summit_description/urdf/summit.urdf.xacro (robot description, xacro)
@@ -495,9 +495,9 @@
      <parent link="base_link"/>
      <child link="camera_link"/>
-     <origin xyz="0.08 0.0 0.265" rpy="0 0 0"/>
+     <origin xyz="0.08 0.07 0.265" rpy="0 0 0"/>
   </joint>
   <link name="camera_link">
     <visual>
-      <origin xyz="0 0 0" rpy="0 0 0"/>
+      <origin xyz="0 -0.07 0" rpy="0 0 0"/>
       <geometry>
         <mesh filename="package://summit_description/meshes/xtion_pro_live.dae" />
@@ -505,5 +505,5 @@
     </visual>
     <collision>
-      <origin xyz="0 0 0" rpy="0 0 0"/>
+      <origin xyz="0 -0.07 0" rpy="0 0 0"/>
       <geometry>
         <mesh filename="package://summit_description/meshes/xtion_pro_live.dae" />

Commit message: Imu added to rviz simulation.

File: summit_sim/summit_description/urdf/summit.urdf.xacro (robot description, xacro)
@@ -512,4 +512,25 @@
   </link>
   <!-- =================================================================== -->
+  <!-- IMU -->
+  <joint name="joint_IMU" type="fixed">
+     <parent link="base_link"/>
+     <child link="imu_link"/>
+     <origin xyz="0.25 0 0.18" rpy="0 0 0"/>
+  </joint>
+  <link name="imu_link">
+    <visual>
+      <origin xyz="0 0 0" rpy="0 0 0"/>
+      <geometry>
+        <box size="0.01 0.01 0.01" />
+      </geometry>
+    </visual>
+    <collision>
+      <origin xyz="0 0 0" rpy="0 0 0"/>
+      <geometry>
+        <box size="0.01 0.01 0.01" />
+      </geometry>
+    </collision>
+  </link>
+  <!-- =================================================================== -->
   <!-- AXIS PTZ CAMERA WITH PAN AND TILT -->
 <!--

Commit message: Added the (Asus) depth_camera TF for simulation.

File: summit_sim/summit_description/urdf/summit.urdf.xacro (robot description, xacro)
@@ -510,5 +510,37 @@
       </geometry>
     </collision>
-  </link>
+    <inertial>
+      <mass value="0.200" />
+      <origin xyz="0 0 0" rpy="0 0 0"/>
+      <inertia ixx="5.8083e-4" ixy="0" ixz="0" iyy="3.0833e-5" iyz="0" izz="5.9083e-4" />
+    </inertial>
+  </link>
+  <!-- depth_frame -->
+  <joint name="camera_depth_joint" type="fixed">
+    <origin xyz="0.0 -0.022 0.0" rpy="0 0 0" />
+    <parent link="camera_link" />
+    <child link="camera_depth_frame"/>
+  </joint>
+   <link name="camera_depth_frame"/>
+   <joint name="camera_depth_optical_joint" type="fixed">
+    <origin xyz="0 0 0" rpy="${-PI/2} 0.0 ${-PI/2}" />
+    <parent link="camera_depth_frame" />
+    <child link="camera_depth_optical_frame"/>
+  </joint>
+   <link name="camera_depth_optical_frame"/>
+   <!-- =================================================================== -->
+  <joint name="camera_rgb_joint" type="fixed">
+    <origin xyz="0.0 -0.049 0.0" rpy="0 0 0" />
+    <parent link="camera_link" />
+    <child link="camera_rgb_frame"/>
+  </joint>
+  <!--  rgb_frame -->
+  <link name="camera_rgb_frame"/>
+  <joint name="camera_rgb_optical_joint" type="fixed">
+    <origin xyz="0 0 0" rpy="${-PI/2} 0.0 ${-PI/2}" />
+    <parent link="camera_rgb_frame" />
+    <child link="camera_rgb_optical_frame"/>
+  </joint>
+   <link name="camera_rgb_optical_frame"/>
   <!-- =================================================================== -->
   <!-- IMU -->

Commit message: Frame to use with the Powerball...

File: summit_sim/summit_description/urdf/summit.urdf.xacro (robot description, xacro)
@@ -564,4 +564,10 @@
     </collision>
   </link>
+  <joint name="to_gripper_joint" type="fixed">
+    <parent link="base_link"/>
+    <child link="to_gripper_link"/>
+    <origin xyz="-0.05 0 0.35" rpy="0 0 0"/>
+  </joint>
+  <link name="to_gripper_link"/>
   <!-- =================================================================== -->
   <!-- AXIS PTZ CAMERA WITH PAN AND TILT -->

Commit message: ultimos cambios de Julian

File: summit_sim/summit_description/urdf/summit.urdf.xacro (robot description, xacro)
@@ -567,5 +567,5 @@
     <parent link="base_link"/>
     <child link="to_gripper_link"/>
-    <origin xyz="-0.05 0 0.35" rpy="0 0 0"/>
+    <origin xyz="-0.08 0 0.6" rpy="0 0 ${PI/2}"/>
   </joint>
   <link name="to_gripper_link"/>
